File: hardware/esp-beep.sch (KiCad schematic (older format))
At the start: 4 parts, among them Q1 J3Y NPN, U1 Wemos_D1_Mini

Commit message: Assign footprints to schematic symbols.
Parts:
- Q1: footprint (none) -> TO_SOT_Packages_SMD:SOT-23_Handsoldering
- R1: footprint (none) -> Resistors_SMD:R_0805_HandSoldering
- SP1: footprint (none) -> CrumpPrints:5V_buzzer
- U1: footprint (none) -> CrumpPrints:D1_mini
Changed lines of the file:
@@
 F 0 "SP1" H 4150 1350 50  0000 C CNN
 F 1 "SPEAKER" H 4150 850 50  0000 C CNN
-F 2 "" H 4250 1100 50  0000 C CNN
+F 2 "CrumpPrints:5V_buzzer" H 4250 1100 50  0001 C CNN
 F 3 "" H 4250 1100 50  0000 C CNN
 	1    4250 1100
@@
 F 0 "Q1" H 4050 1700 50  0000 R CNN
 F 1 "J3Y NPN" H 4250 1600 50  0000 R CNN
-F 2 "" H 3950 1750 50  0000 C CNN
+F 2 "TO_SOT_Packages_SMD:SOT-23_Handsoldering" H 3950 1750 50  0001 C CNN
 F 3 "" H 3750 1650 50  0000 C CNN
 	1    3750 1650
@@
 F 0 "R1" V 3250 1600 50  0000 L CNN
 F 1 "2.2K" V 3450 1600 50  0000 L CNN
-F 2 "" H 3350 1650 50  0000 C CNN
+F 2 "Resistors_SMD:R_0805_HandSoldering" H 3350 1650 50  0001 C CNN
 F 3 "" H 3350 1650 50  0000 C CNN
 	1    3350 1650
@@
 F 0 "U1" H 1600 600 60  0000 C CNN
 F 1 "Wemos_D1_Mini" H 1600 1700 60  0000 C CNN
-F 2 "" H 1600 1300 60  0001 C CNN
+F 2 "CrumpPrints:D1_mini" H 1600 1300 60  0001 C CNN
 F 3 "" H 1600 1300 60  0001 C CNN
 	1    1600 1300
@@
 NoConn ~ 1050 1400
 $Comp
-L PWR_FLAG #FLG?
+L PWR_FLAG #FLG01
 U 1 1 58E1D111
 P 2750 1200
-F 0 "#FLG?" H 2750 1295 50  0001 C CNN
+F 0 "#FLG01" H 2750 1295 50  0001 C CNN
 F 1 "PWR_FLAG" H 2750 1380 50  0000 C CNN
 F 2 "" H 2750 1200 50  0000 C CNN
@@
 $EndComp
 $Comp
-L PWR_FLAG #FLG?
+L PWR_FLAG #FLG02
 U 1 1 58E1D12D
 P 3150 1200
-F 0 "#FLG?" H 3150 1295 50  0001 C CNN
+F 0 "#FLG02" H 3150 1295 50  0001 C CNN
 F 1 "PWR_FLAG" H 3150 1380 50  0000 C CNN
 F 2 "" H 3150 1200 50  0000 C CNN
